File: pcb/bakeneko-65-pcb.kicad_pcb (KiCad board)
At the start: 2 copper layers, 303.8 x 94.2 mm, 161 parts, among them J1 JST SH 4-pin, J2 AVR-ISP-6, SW1 Reset, U1 SRV05-4, U2 ATmega32U4-AU, Y1 16MHz

Commit message: agrega sockets
Parts:
- MX1, MX10, MX11, MX12, MX13, MX14, MX15, MX16, MX19, MX2, MX20, MX21, MX22, MX23, MX24, MX25, MX26, MX27, MX28, MX29, MX3, MX30, MX32, MX35, MX36, MX37, MX38, MX39, MX4, MX40, MX41, MX42, MX43, MX44, MX45, MX47, MX49, MX5, MX50, MX51, MX52, MX53, MX54, MX55, MX56, MX57, MX58, MX6, MX60, MX61, MX63, MX68, MX69, MX7, MX70, MX8, MX9: value 1u -> MX-NoLED; footprint MX_Only:MXOnly-1U-NoLED -> kbd:CherryMX_Hotswap
- MX17: value 2u -> MX-NoLED; footprint MX_Only:MXOnly-2U-NoLED -> kbd:CherryMX_Hotswap
- MX18, MX31, MX62, MX64, MX67: value 1.5u -> MX-NoLED; footprint MX_Only:MXOnly-1.5U-NoLED -> kbd:CherryMX_Hotswap
- MX33, MX66, MX71, MX72, MX73, MX75: value 1.25u -> MX-NoLED; footprint MX_Only:MXOnly-1.25U-NoLED -> kbd:CherryMX_Hotswap
- MX34, MX59: value 1.75u -> MX-NoLED; footprint MX_Only:MXOnly-1.75U-NoLED -> kbd:CherryMX_Hotswap
- MX46, MX48: value 2.25u -> MX-NoLED; footprint MX_Only:MXOnly-2.25U-NoLED -> kbd:CherryMX_Hotswap
- MX65: value 7u -> MX-NoLED; footprint MX_Only:MXOnly-7U-ReversedStabilizers-NoLED -> kbd:CherryMX_Hotswap
- MX74: value 6.25u -> MX-NoLED; footprint MX_Only:MXOnly-6.25U-ReversedStabilizers-NoLED -> kbd:CherryMX_Hotswap
- moved F1 167.0 mm to (177.3, 85.1)
- moved R3 161.7 mm to (177.3, 87.8)
- moved R2 161.5 mm to (177.3, 89.8)
- moved C2 160.2 mm to (173.1, 75.4), turned to 270 degrees
- moved U1 160.1 mm to (181.5, 88.8)
- moved C4 158.3 mm to (170.1, 87.5), turned to 0 degrees
- moved C7 149.5 mm to (164.7, 88.4), turned to 0 degrees
- moved U2 142.5 mm to (164.8, 79.5), turned to 90 degrees
- moved J1 140.9 mm to (187.6, 88.8)
- moved R4 140.9 mm to (169.8, 71.4), turned to 180 degrees
- moved C3 129.1 mm to (155.0, 86.5), turned to 180 degrees
- moved C1 129.1 mm to (160.7, 71.4), turned to 180 degrees
- moved C5 122.1 mm to (153.1, 83.2)
- moved R1 120.1 mm to (156.9, 88.6), turned to 180 degrees
- moved Y1 119.8 mm to (153.1, 79.8), turned to 270 degrees
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Connections:
- MX1 pad 1: Net-(D1-Pad2) -> COL0
- MX1 pad 2: COL0 -> Net-(D1-Pad2)
- MX10 pad 1: Net-(D10-Pad2) -> COL9
- MX10 pad 2: COL9 -> Net-(D10-Pad2)
- MX11 pad 1: Net-(D11-Pad2) -> COL10
- MX11 pad 2: COL10 -> Net-(D11-Pad2)
- MX12 pad 1: Net-(D12-Pad2) -> COL11
- MX12 pad 2: COL11 -> Net-(D12-Pad2)
- MX13 pad 1: Net-(D13-Pad2) -> COL12
- MX13 pad 2: COL12 -> Net-(D13-Pad2)
- MX14 pad 1: Net-(D14-Pad2) -> COL13
- MX14 pad 2: COL13 -> Net-(D14-Pad2)
- MX15 pad 1: Net-(D15-Pad2) -> COL14
- MX15 pad 2: COL14 -> Net-(D15-Pad2)
- MX16 pad 1: Net-(D16-Pad2) -> COL15
- MX16 pad 2: COL15 -> Net-(D16-Pad2)
- MX17 pad 1: Net-(D15-Pad2) -> COL14
- MX17 pad 2: COL14 -> Net-(D15-Pad2)
- MX18 pad 1: Net-(D17-Pad2) -> COL0
- MX18 pad 2: COL0 -> Net-(D17-Pad2)
- MX19 pad 1: Net-(D18-Pad2) -> COL1
- MX19 pad 2: COL1 -> Net-(D18-Pad2)
- MX2 pad 1: Net-(D2-Pad2) -> COL1
- MX2 pad 2: COL1 -> Net-(D2-Pad2)
- MX20 pad 1: Net-(D19-Pad2) -> COL2
- MX20 pad 2: COL2 -> Net-(D19-Pad2)
- MX21 pad 1: Net-(D20-Pad2) -> COL3
- MX21 pad 2: COL3 -> Net-(D20-Pad2)
- MX22 pad 1: Net-(D21-Pad2) -> COL4
- MX22 pad 2: COL4 -> Net-(D21-Pad2)
- MX23 pad 1: Net-(D22-Pad2) -> COL5
- MX23 pad 2: COL5 -> Net-(D22-Pad2)
- MX24 pad 1: Net-(D23-Pad2) -> COL6
- MX24 pad 2: COL6 -> Net-(D23-Pad2)
- MX25 pad 1: Net-(D24-Pad2) -> COL7
- MX25 pad 2: COL7 -> Net-(D24-Pad2)
- MX26 pad 1: Net-(D25-Pad2) -> COL8
- MX26 pad 2: COL8 -> Net-(D25-Pad2)
- MX27 pad 1: Net-(D26-Pad2) -> COL9
- MX27 pad 2: COL9 -> Net-(D26-Pad2)
- MX28 pad 1: Net-(D27-Pad2) -> COL10
- MX28 pad 2: COL10 -> Net-(D27-Pad2)
- MX29 pad 1: Net-(D28-Pad2) -> COL11
- MX29 pad 2: COL11 -> Net-(D28-Pad2)
- MX3 pad 1: Net-(D3-Pad2) -> COL2
- MX3 pad 2: COL2 -> Net-(D3-Pad2)
- MX30 pad 1: Net-(D29-Pad2) -> COL12
- MX30 pad 2: COL12 -> Net-(D29-Pad2)
- MX31 pad 1: Net-(D30-Pad2) -> COL13
- MX31 pad 2: COL13 -> Net-(D30-Pad2)
- MX32 pad 1: Net-(D31-Pad2) -> COL15
- MX32 pad 2: COL15 -> Net-(D31-Pad2)
- MX33 pad 1: Net-(D32-Pad2) -> COL0
- MX33 pad 2: COL0 -> Net-(D32-Pad2)
- MX34 pad 1: Net-(D32-Pad2) -> COL0
- MX34 pad 2: COL0 -> Net-(D32-Pad2)
- MX35 pad 1: Net-(D33-Pad2) -> COL1
- MX35 pad 2: COL1 -> Net-(D33-Pad2)
- MX36 pad 1: Net-(D34-Pad2) -> COL2
- MX36 pad 2: COL2 -> Net-(D34-Pad2)
- MX37 pad 1: Net-(D35-Pad2) -> COL3
- MX37 pad 2: COL3 -> Net-(D35-Pad2)
- MX38 pad 1: Net-(D36-Pad2) -> COL4
- MX38 pad 2: COL4 -> Net-(D36-Pad2)
- MX39 pad 1: Net-(D37-Pad2) -> COL5
- MX39 pad 2: COL5 -> Net-(D37-Pad2)
- MX4 pad 1: Net-(D4-Pad2) -> COL3
- MX4 pad 2: COL3 -> Net-(D4-Pad2)
- MX40 pad 1: Net-(D38-Pad2) -> COL6
- MX40 pad 2: COL6 -> Net-(D38-Pad2)
- MX41 pad 1: Net-(D39-Pad2) -> COL7
- MX41 pad 2: COL7 -> Net-(D39-Pad2)
- MX42 pad 1: Net-(D40-Pad2) -> COL8
- MX42 pad 2: COL8 -> Net-(D40-Pad2)
- MX43 pad 1: Net-(D41-Pad2) -> COL9
- MX43 pad 2: COL9 -> Net-(D41-Pad2)
- MX44 pad 1: Net-(D42-Pad2) -> COL10
- MX44 pad 2: COL10 -> Net-(D42-Pad2)
- MX45 pad 1: Net-(D43-Pad2) -> COL11
- MX45 pad 2: COL11 -> Net-(D43-Pad2)
- MX46 pad 1: Net-(D44-Pad2) -> COL13
- MX46 pad 2: COL13 -> Net-(D44-Pad2)
- MX47 pad 1: Net-(D45-Pad2) -> COL15
- MX47 pad 2: COL15 -> Net-(D45-Pad2)
- MX48 pad 1: Net-(D46-Pad2) -> COL0
- MX48 pad 2: COL0 -> Net-(D46-Pad2)
- MX49 pad 1: Net-(D47-Pad2) -> COL2
- MX49 pad 2: COL2 -> Net-(D47-Pad2)
- MX5 pad 1: Net-(D5-Pad2) -> COL4
- MX5 pad 2: COL4 -> Net-(D5-Pad2)
- MX50 pad 1: Net-(D48-Pad2) -> COL3
- MX50 pad 2: COL3 -> Net-(D48-Pad2)
- MX51 pad 1: Net-(D49-Pad2) -> COL4
- MX51 pad 2: COL4 -> Net-(D49-Pad2)
- MX52 pad 1: Net-(D50-Pad2) -> COL5
- MX52 pad 2: COL5 -> Net-(D50-Pad2)
- MX53 pad 1: Net-(D51-Pad2) -> COL6
- MX53 pad 2: COL6 -> Net-(D51-Pad2)
- MX54 pad 1: Net-(D52-Pad2) -> COL7
- MX54 pad 2: COL7 -> Net-(D52-Pad2)
- MX55 pad 1: Net-(D53-Pad2) -> COL8
- MX55 pad 2: COL8 -> Net-(D53-Pad2)
- MX56 pad 1: Net-(D54-Pad2) -> COL9
- MX56 pad 2: COL9 -> Net-(D54-Pad2)
- MX57 pad 1: Net-(D55-Pad2) -> COL10
- MX57 pad 2: COL10 -> Net-(D55-Pad2)
- MX58 pad 1: Net-(D56-Pad2) -> COL11
- MX58 pad 2: COL11 -> Net-(D56-Pad2)
- MX59 pad 1: Net-(D57-Pad2) -> COL12
- MX59 pad 2: COL12 -> Net-(D57-Pad2)
- MX6 pad 1: Net-(D6-Pad2) -> COL5
- MX6 pad 2: COL5 -> Net-(D6-Pad2)
- MX60 pad 1: Net-(D58-Pad2) -> COL13
- MX60 pad 2: COL13 -> Net-(D58-Pad2)
- MX61 pad 1: Net-(D59-Pad2) -> COL15
- MX61 pad 2: COL15 -> Net-(D59-Pad2)
- MX62 pad 1: Net-(D60-Pad2) -> COL0
- MX62 pad 2: COL0 -> Net-(D60-Pad2)
- MX63 pad 1: Net-(D61-Pad2) -> COL1
- MX63 pad 2: COL1 -> Net-(D61-Pad2)
- MX64 pad 1: Net-(D62-Pad2) -> COL2
- MX64 pad 2: COL2 -> Net-(D62-Pad2)
- MX65 pad 1: Net-(D63-Pad2) -> COL6
- MX65 pad 2: COL6 -> Net-(D63-Pad2)
- MX66 pad 1: Net-(D64-Pad2) -> COL9
- MX66 pad 2: COL9 -> Net-(D64-Pad2)
- MX67 pad 1: Net-(D65-Pad2) -> COL11
- MX67 pad 2: COL11 -> Net-(D65-Pad2)
- MX68 pad 1: Net-(D66-Pad2) -> COL12
- MX68 pad 2: COL12 -> Net-(D66-Pad2)
- MX69 pad 1: Net-(D67-Pad2) -> COL13
- MX69 pad 2: COL13 -> Net-(D67-Pad2)
- MX7 pad 1: Net-(D7-Pad2) -> COL6
- MX7 pad 2: COL6 -> Net-(D7-Pad2)
- MX70 pad 1: Net-(D68-Pad2) -> COL15
- MX70 pad 2: COL15 -> Net-(D68-Pad2)
- MX71 pad 1: Net-(D60-Pad2) -> COL0
- MX71 pad 2: COL0 -> Net-(D60-Pad2)
- MX72 pad 1: Net-(D61-Pad2) -> COL1
- MX72 pad 2: COL1 -> Net-(D61-Pad2)
- MX73 pad 1: Net-(D62-Pad2) -> COL2
- MX73 pad 2: COL2 -> Net-(D62-Pad2)
- MX74 pad 1: Net-(D63-Pad2) -> COL6
- MX74 pad 2: COL6 -> Net-(D63-Pad2)
- MX75 pad 1: Net-(D65-Pad2) -> COL11
- MX75 pad 2: COL11 -> Net-(D65-Pad2)
- MX8 pad 1: Net-(D8-Pad2) -> COL7
- MX8 pad 2: COL7 -> Net-(D8-Pad2)
- MX9 pad 1: Net-(D9-Pad2) -> COL8
- MX9 pad 2: COL8 -> Net-(D9-Pad2)
- U1 pad 3: Net-(U1-Pad3) -> (no net)
- U1 pad 4: Net-(U1-Pad4) -> (no net)
- U2 pad 1: ROW0 -> (no net)
- U2 pad 12: ROW1 -> COL6
- U2 pad 18: COL15 -> COL1
- U2 pad 19: COL14 -> COL2
- U2 pad 20: COL13 -> COL3
- U2 pad 21: COL12 -> COL4
- U2 pad 22: COL11 -> COL5
- U2 pad 25: COL10 -> COL7
- U2 pad 26: COL9 -> ROW3
- U2 pad 28: COL7 -> ROW0
- U2 pad 29: COL6 -> ROW2
- U2 pad 30: COL5 -> ROW1
- U2 pad 31: COL4 -> COL9
- U2 pad 32: COL3 -> COL10
- U2 pad 36: ROW2 -> COL11
- U2 pad 37: COL0 -> COL12
- U2 pad 38: ROW4 -> COL13
- U2 pad 39: ROW3 -> COL14
- U2 pad 40: COL2 -> COL15
- U2 pad 41: Net-(U2-Pad41) -> ROW4
- U2 pad 42: Net-(U2-Pad42) -> (no net)
- U2 pad 8: COL1 -> COL0
Routing:
- net COL0: track 99.8 -> 265.8 mm, vias 1 -> 8
- net COL13: track 353.1 -> 195.9 mm, vias 0 -> 8
- net COL11: track 293.6 -> 138.0 mm, vias 0 -> 8
- net COL15: track 355.0 -> 199.4 mm, vias 0 -> 8
- net COL12: track 318.3 -> 163.3 mm, vias 0 -> 6
- net COL10: track 254.7 -> 102.2 mm, vias 0 -> 6
- net COL9: track 266.7 -> 117.9 mm, vias 0 -> 8
- net ROW0: track 295.7 -> 439.9 mm
- net ROW1: track 284.9 -> 422.7 mm
- net COL8: track 217.4 -> 81.5 mm, vias 0 -> 6
- net COL14: track 318.9 -> 207.8 mm, vias 1 -> 2
- net COL1: track 113.8 -> 213.1 mm, vias 0 -> 7
- net COL7: track 198.8 -> 100.4 mm, vias 0 -> 6
- net ROW2: track 301.5 -> 387.7 mm
- net COL6: track 212.1 -> 139.8 mm, vias 0 -> 10
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Other:
- net class Default: trace_width 0.25 -> 0.254
