File: pcb/bakeneko-65-pcb.sch (KiCad schematic (older format))
At the start: 18 parts, among them J1 JST SH 4-pin, J2 AVR-ISP-6, SW1 Reset, U1 SRV05-4, U2 ATmega32U4-AU, Y1 16MHz

Commit message: agrega sockets
Parts:
- J2: symbol Connector:AVR-ISP-6 -> bakeneko-65-pcb-rescue:AVR-ISP-6-Connector
- U2: symbol MCU_Microchip_ATmega:ATmega32U4-AU -> bakeneko-65-pcb-rescue:ATmega32U4-AU-MCU_Microchip_ATmega
Connections:
- no-connect marks 4 -> 3
Changed lines of the file:
@@
 EESchema Schematic File Version 4
-LIBS:bakeneko-65-pcb-cache
 EELAYER 30 0
 EELAYER END
@@
 D+
 $Comp
-L MCU_Microchip_ATmega:ATmega32U4-AU U2
-U 1 1 5F26004F
-P 2350 5400
-F 0 "U2" H 1500 4550 50  0000 C CNN
-F 1 "ATmega32U4-AU" H 1500 4450 50  0000 C CNN
-F 2 "Package_QFP:TQFP-44_10x10mm_P0.8mm" H 2350 5400 50  0001 C CIN
-F 3 "http://ww1.microchip.com/downloads/en/DeviceDoc/Atmel-7766-8-bit-AVR-ATmega16U4-32U4_Datasheet.pdf" H 2350 5400 50  0001 C CNN
-F 4 "C44854" H 2350 5400 50  0001 C CNN "LCSC Part #"
-	1    2350 5400
-	1    0    0    -1
-$EndComp
-$Comp
 L Device:R R3
 U 1 1 5F259605
@@
 	1    0    0    -1
 $EndComp
-Wire Wire Line
-	1500 5200 1750 5200
 $Comp
 L power:GND #PWR022
@@
 	5050 5400 5500 5400
 $Comp
-L Connector:AVR-ISP-6 J2
+L bakeneko-65-pcb-rescue:AVR-ISP-6-Connector J2
 U 1 1 5F4C9CCE
 P 4600 1650
@@
 Text GLabel 2950 4100 2    50   Input ~ 0
 MOSI
-Text GLabel 2950 5100 2    50   Input ~ 0
-COL15
-Text GLabel 2950 5200 2    50   Input ~ 0
-COL14
-Text GLabel 2950 5300 2    50   Input ~ 0
-COL13
-Text GLabel 2950 5400 2    50   Input ~ 0
-COL12
-Text GLabel 2950 5600 2    50   Input ~ 0
-COL11
-Text GLabel 2950 5500 2    50   Input ~ 0
-COL10
-Text GLabel 2950 5700 2    50   Input ~ 0
-COL9
-Text GLabel 2950 5800 2    50   Input ~ 0
-COL8
-Text GLabel 2950 4300 2    50   Input ~ 0
-COL7
-Text GLabel 2950 4400 2    50   Input ~ 0
-COL6
-Text GLabel 2950 4500 2    50   Input ~ 0
-COL5
-Text GLabel 2950 4800 2    50   Input ~ 0
-COL4
-Text GLabel 2950 3900 2    50   Input ~ 0
-COL1
-Text GLabel 2950 6700 2    50   Input ~ 0
-COL0
-Text GLabel 2950 4600 2    50   Input ~ 0
-ROW1
-Text GLabel 2950 6800 2    50   Input ~ 0
-ROW2
-Text GLabel 2950 6100 2    50   Input ~ 0
-ROW0
 Wire Wire Line
 	5400 3800 5400 3650
@@
 	5400 4250 5400 4100
 Connection ~ 5000 4250
-Text GLabel 2950 4900 2    50   Input ~ 0
-COL3
-NoConn ~ 2950 6300
 $Comp
 L power:GND #PWR02
@@
 F1 "matrix.sch" 50
 $EndSheet
-Wire Wire Line
-	2150 3600 2250 3600
-Wire Wire Line
-	2150 7200 2250 7200
-Wire Wire Line
-	2350 3600 2450 3600
-Wire Wire Line
-	2250 3600 2350 3600
-Connection ~ 2250 3600
-Connection ~ 2350 3600
-Wire Wire Line
-	2350 7200 2250 7200
-Connection ~ 2250 7200
 $Comp
 L power:+5V #PWR0107
@@
 	0    -1   -1   0
 $EndComp
-Wire Wire Line
-	1250 4900 1750 4900
-Wire Wire Line
-	1250 5000 1750 5000
 Text Label 1350 4900 0    50   ~ 0
 MCU_D+
 Text Label 1350 5000 0    50   ~ 0
 MCU_D-
-Text GLabel 2950 6400 2    50   Input ~ 0
-COL2
-Text GLabel 2950 6600 2    50   Input ~ 0
-ROW4
-Text GLabel 2950 6500 2    50   Input ~ 0
-ROW3
 $Comp
 L Power_Protection:SRV05-4 U1
@@
 Wire Wire Line
 	6150 2800 6000 2800
+Connection ~ 2250 7200
+Connection ~ 2250 3600
+Connection ~ 2350 3600
+Text GLabel 2950 6300 2    50   Input ~ 0
+ROW4
+Wire Wire Line
+	1500 5200 1750 5200
+Wire Wire Line
+	2150 7200 2250 7200
+Wire Wire Line
+	1250 4900 1750 4900
+Wire Wire Line
+	1250 5000 1750 5000
+Wire Wire Line
+	2350 3600 2450 3600
+Wire Wire Line
+	2150 3600 2250 3600
+Wire Wire Line
+	2350 7200 2250 7200
+Wire Wire Line
+	2250 3600 2350 3600
+$Comp
+L bakeneko-65-pcb-rescue:ATmega32U4-AU-MCU_Microchip_ATmega U2
+U 1 1 5F26004F
+P 2350 5400
+F 0 "U2" H 1500 4550 50  0000 C CNN
+F 1 "ATmega32U4-AU" H 1500 4450 50  0000 C CNN
+F 2 "Package_QFP:TQFP-44_10x10mm_P0.8mm" H 2350 5400 50  0001 C CIN
+F 3 "http://ww1.microchip.com/downloads/en/DeviceDoc/Atmel-7766-8-bit-AVR-ATmega16U4-32U4_Datasheet.pdf" H 2350 5400 50  0001 C CNN
+F 4 "C44854" H 2350 5400 50  0001 C CNN "LCSC Part #"
+	1    2350 5400
+	1    0    0    -1
+$EndComp
+Text GLabel 2950 3900 2    50   Input ~ 0
+COL0
+Text GLabel 2950 5100 2    50   Input ~ 0
+COL1
+Text GLabel 2950 5200 2    50   Input ~ 0
+COL2
+Text GLabel 2950 5300 2    50   Input ~ 0
+COL3
+Text GLabel 2950 5400 2    50   Input ~ 0
+COL4
+Text GLabel 2950 5600 2    50   Input ~ 0
+COL5
+Text GLabel 2950 4600 2    50   Input ~ 0
+COL6
+Text GLabel 2950 5700 2    50   Input ~ 0
+ROW3
+Text GLabel 2950 5800 2    50   Input ~ 0
+COL8
+Text GLabel 2950 4300 2    50   Input ~ 0
+ROW0
+Text GLabel 2950 4400 2    50   Input ~ 0
+ROW2
+Text GLabel 2950 4500 2    50   Input ~ 0
+ROW1
+Text GLabel 2950 4800 2    50   Input ~ 0
+COL9
+Text GLabel 2950 6400 2    50   Input ~ 0
+COL15
+Text GLabel 2950 6500 2    50   Input ~ 0
+COL14
+Text GLabel 2950 6600 2    50   Input ~ 0
+COL13
+Text GLabel 2950 6700 2    50   Input ~ 0
+COL12
+Text GLabel 2950 6800 2    50   Input ~ 0
+COL11
+Text GLabel 2950 4900 2    50   Input ~ 0
+COL10
+Text GLabel 2950 5500 2    50   Input ~ 0
+COL7
 $EndSCHEMATC
