File: pcb/matrix.sch (KiCad schematic (older format))
At the start: 143 parts

Commit message: agrega sockets
Parts:
- removed MX1, MX10, MX11, MX12, MX13, MX14, MX15, MX16, MX19, MX2, MX20, MX21, MX22, MX23, MX24, MX25, MX26, MX27, MX28, MX29, MX3, MX30, MX32, MX35, MX36, MX37, MX38, MX39, MX4, MX40, MX41, MX42, MX43, MX44, MX45, MX47, MX49, MX5, MX50, MX51, MX52, MX53, MX54, MX55, MX56, MX57, MX58, MX6, MX60, MX61, MX63, MX68, MX69, MX7, MX70, MX8, MX9: 1u, MX_Only:MXOnly-1U-NoLED, symbol Switch:SW_SPST
- removed MX17: 2u, MX_Only:MXOnly-2U-NoLED, symbol Switch:SW_SPST
- removed MX18, MX31, MX62, MX64, MX67: 1.5u, MX_Only:MXOnly-1.5U-NoLED, symbol Switch:SW_SPST
- removed MX33, MX66, MX71, MX72, MX73, MX75: 1.25u, MX_Only:MXOnly-1.25U-NoLED, symbol Switch:SW_SPST
- removed MX34, MX59: 1.75u, MX_Only:MXOnly-1.75U-NoLED, symbol Switch:SW_SPST
- removed MX46, MX48: 2.25u, MX_Only:MXOnly-2.25U-NoLED, symbol Switch:SW_SPST
- removed MX65: 7u, MX_Only:MXOnly-7U-ReversedStabilizers-NoLED, symbol Switch:SW_SPST
- removed MX74: 6.25u, MX_Only:MXOnly-6.25U-ReversedStabilizers-NoLED, symbol Switch:SW_SPST
- added MX1, MX10, MX11, MX12, MX13, MX14, MX15, MX16, MX17, MX18, MX19, MX2, MX20, MX21, MX22, MX23, MX24, MX25, MX26, MX27, MX28, MX29, MX3, MX30, MX31, MX32, MX33, MX34, MX35, MX36, MX37, MX38, MX39, MX4, MX40, MX41, MX42, MX43, MX44, MX45, MX46, MX47, MX48, MX49, MX5, MX50, MX51, MX52, MX53, MX54, MX55, MX56, MX57, MX58, MX59, MX6, MX60, MX61, MX62, MX63, MX64, MX65, MX66, MX67, MX68, MX69, MX7, MX70, MX71, MX72, MX73, MX74, MX75, MX8, MX9: MX-NoLED, kbd:CherryMX_Hotswap, symbol MX_Alps_Hybrid:MX-NoLED
Connections:
- wire segments 168 -> 170
Other:
- moved on the sheet: D1, D10, D11, D12, D13, D14, D15, D16, D17, D18, D19, D2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
